File: mainboard/main.sch (EAGLE design)
At the start: 4 parts, among them J1 RJHSE-3380, J2 RJHSE-3380, J3 RJHSE-3380

Commit message: main v2
Parts:
- removed J1, J2, J3: RJHSE-3380, RJHSE-3380:RJHSE-3380
- added C2, CPV2, LEGACY: RA-RJ45RA, comma.ai:RA-RJ45RA
- added OPTION: 34793-0041, 34793-0041:34793-0041
Connections:
- net CAN0_H: now also C2.6, CPV2.6, LEGACY.6; no longer J2.6, J3.6
- net CAN0_L: now also C2.3, CPV2.3, LEGACY.3; no longer J2.3, J3.3
- net CAN1_H: now also OPTION.1, OPTION.3; no longer J1.4
- net CAN1_L: now also OPTION.2, OPTION.4; no longer J1.5
- net CAN2_H: now also C2.4, CPV2.4; no longer J1.2, J2.4, J3.4
- net CAN2_L: now also C2.2, CPV2.2; no longer J1.3, J2.2, J3.2
- net GND: now also C2.1, C2.5, C2.P$1, C2.P$2, CPV2.1, CPV2.5, CPV2.P$1, CPV2.P$2, LEGACY.1, LEGACY.5, LEGACY.P$1, LEGACY.P$2; no longer J1.7, J1.8, J2.1, J2.5, J3.1, J3.5
- net VIN: now also C2.7, C2.8, CPV2.7, CPV2.8, LEGACY.2; no longer J1.1, J1.6, J2.7, J2.8, J3.7, J3.8
Other:
- note added: "CAN0 - car harness CAN0 CAN1 - B-CAN CAN2 - OBD2 F-CAN-A"
- note removed: "CAN0 - car harness CAN0 CAN1 - B-CAN CAN2 - F-CAN-A/OBD2 F-CAN-A"
