File: board/main.brd (EAGLE design)
At the start: 76.3 x 39.4 mm, 5 parts

Commit message: rev1.1c push and cleanup
Parts:
- moved OPTION 1.27 mm to (44.6, 12.4)
Connections:
- net CAN1_H: no longer OPTION.3
- net CAN1_L: no longer OPTION.4
- net K_LINE: now also OPTION.3
- net L_LINE: now also OPTION.4
- net VIN: no longer LEGACY.2
Routing:
- net L_LINE: track 0.00 -> 31.4 mm, vias 0 -> 1
- net K_LINE: track 0.00 -> 27.1 mm, vias 0 -> 2
- net VIN: track 82.7 -> 77.0 mm
- net CAN1_L: track 26.0 -> 22.0 mm
- net CAN1_H: track 48.0 -> 44.1 mm
- net GND: track 247.7 -> 248.9 mm, vias 6 -> 8
Other:
- board text added: "csouers 01/13/2021"
- board text added: "rev 1.1"
- board text removed: "csouers 8/18/2020"
