File: board/main.sch (EAGLE design)
At the start: 5 parts

Commit message: rev1.1c push and cleanup
Connections:
- net CAN1_H: no longer OPTION.3
- net CAN1_L: no longer OPTION.4
- net K_LINE: now also OPTION.3
- net L_LINE: now also OPTION.4
- net VIN: no longer LEGACY.2
Changed lines of the file:
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@@
 </variantdefs>
 <classes>
-<class number="0" name="default" width="0.3048" drill="0">
+<class number="0" name="default" width="0.508" drill="0">
 </class>
 <class number="1" name="PWR" width="0.8128" drill="0">
@@
 <label x="2.54" y="7.62" size="1.778" layer="95"/>
 </segment>
+<segment>
+<pinref part="OPTION" gate="G$1" pin="4"/>
+<wire x1="22.86" y1="66.04" x2="20.32" y2="66.04" width="0.1524" layer="91"/>
+<label x="20.32" y="66.04" size="1.778" layer="95" rot="R180"/>
+</segment>
 </net>
 <net name="K_LINE" class="0">
@@
 <label x="-53.34" y="7.62" size="1.778" layer="95" rot="R180"/>
 </segment>
+<segment>
+<pinref part="OPTION" gate="G$1" pin="3"/>
+<wire x1="22.86" y1="68.58" x2="20.32" y2="68.58" width="0.1524" layer="91"/>
+<label x="20.32" y="68.58" size="1.778" layer="95" rot="R180"/>
+</segment>
 </net>
 <net name="IGN" class="1">
@@
 </segment>
 <segment>
-<pinref part="LEGACY" gate="G$1" pin="2"/>
-<wire x1="-30.48" y1="88.9" x2="-33.02" y2="88.9" width="0.1524" layer="91"/>
-<label x="-33.02" y="88.9" size="1.778" layer="95" rot="R180"/>
-</segment>
-<segment>
 <pinref part="C2" gate="G$1" pin="7"/>
 <wire x1="-83.82" y1="48.26" x2="-86.36" y2="48.26" width="0.1524" layer="91"/>
@@
 <label x="20.32" y="73.66" size="1.778" layer="95" rot="R180"/>
 </segment>
-<segment>
-<pinref part="OPTION" gate="G$1" pin="3"/>
-<wire x1="22.86" y1="68.58" x2="20.32" y2="68.58" width="0.1524" layer="91"/>
-<label x="20.32" y="68.58" size="1.778" layer="95" rot="R180"/>
-</segment>
 </net>
 <net name="GMLAN" class="0">
@@
 <label x="20.32" y="71.12" size="1.778" layer="95" rot="R180"/>
 </segment>
-<segment>
-<pinref part="OPTION" gate="G$1" pin="4"/>
-<wire x1="22.86" y1="66.04" x2="20.32" y2="66.04" width="0.1524" layer="91"/>
-<label x="20.32" y="66.04" size="1.778" layer="95" rot="R180"/>
-</segment>
 </net>
 </nets>
 </sheet>
 </sheets>
+<errors>
+</errors>
 </schematic>
 </drawing>
